File: HALMET.kicad_sch (KiCad schematic)
At the start: 0 parts

Commit message: HALMET redesign
Other:
- removed sheet Optocouplers
- added sheet Analog input (analog_input.kicad_sch)
- added sheet Digital input (digital_input.kicad_sch)
- added sheet Isolation barrier (isolation.kicad_sch)
- sheet CAN bus ports: added CAN_H, CAN_L; removed none
- sheet ESP32 ports: added DI1, DI2, DI3, DI4, IO2; removed LED, OPTO_IN1, OPTO_OUT1
- sheet Power input ports: added CAN_H, CAN_L; removed none
- sheet User Interface ports: added CAN_RX, CAN_TX; removed none
- title: Sailor Hat with ESP32 -> Hat Labs Marine Engine/Tank interface (HALMET)

Commit message: Implement HALMET v1.0.0 design changes
Other:
- title: Hat Labs Marine Engine/Tank interface (HALMET) -> Hat Labs Marine Engine & Tank interface (HALMET)
Changed lines of the file:
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@@
   (paper "A4")
   (title_block
-    (title "Hat Labs Marine Engine/Tank interface (HALMET)")
-    (date "2023-09-19")
-    (rev "1.0.0-a1")
+    (title "Hat Labs Marine Engine & Tank interface (HALMET)")
+    (date "2023-11-27")
+    (rev "1.0.0")
     (company "Hat Labs Ltd")
     (comment 1 "https://creativecommons.org/licenses/by-sa/4.0")

Commit message: Fix DI4 & DI3 pins
Changed lines of the file:
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@@
+    (stroke (width 0) (type default))
+  )
+  (wire (pts (xy 156.21 91.44) (xy 158.75 91.44))
+    (stroke (width 0) (type default))
+  )
+  (wire (pts (xy 233.68 39.37) (xy 236.22 39.37))
     (stroke (width 0) (type default))
   )
   (wire (pts (xy 156.21 87.63) (xy 158.75 87.63))
-    (stroke (width 0) (type default))
-  )
-  (wire (pts (xy 233.68 39.37) (xy 236.22 39.37))
-    (stroke (width 0) (type default))
-  )
-  (wire (pts (xy 156.21 91.44) (xy 158.75 91.44))
     (stroke (width 0) (type default))
   )
@@
       (effects (font (size 1.27 1.27)) (justify right))
     )
-    (pin "DI4" input (at 156.21 87.63 0)
-      (effects (font (size 1.27 1.27)) (justify right))
-    )
-    (pin "DI3" input (at 156.21 91.44 0)
-      (effects (font (size 1.27 1.27)) (justify right))
-    )
+    (pin "DI4" input (at 156.21 91.44 0)
+      (effects (font (size 1.27 1.27)) (justify right))
+    )
+    (pin "DI3" input (at 156.21 87.63 0)
+      (effects (font (size 1.27 1.27)) (justify right))
+    )
