File: UI.kicad_sch (KiCad schematic)
At the start: 8 parts, among them SW501 SW_Push, SW502 SW_Push

Commit message: HALMET redesign
Parts:
- added D1001, D1002: GREEN LED, LED_SMD:LED_0603_1608Metric, symbol Device:LED
- added R1001, R1002: 1.5k, Resistor_SMD:R_0402_1005Metric, symbol Device:R
Connections:
- net +3V3 renamed +3.3V
- net +3.3V: now also R1001.1, R1002.1
- new net: D1002.2 (A), R1002.2
- new net: D1001.2 (A), R1001.2
- new net CAN_RX: D1001.1 (K)
- new net CAN_TX: D1002.1 (K)
Other:
- title: Sailor Hat with ESP32 -> Hat Labs Marine Engine/Tank interface (HALMET)

Commit message: Implement HALMET v1.0.0 design changes
Other:
- title: Hat Labs Marine Engine/Tank interface (HALMET) -> Hat Labs Marine Engine & Tank interface (HALMET)
Changed lines of the file:
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@@
   (paper "A4")
   (title_block
-    (title "Hat Labs Marine Engine/Tank interface (HALMET)")
-    (date "2023-09-19")
-    (rev "1.0.0-a1")
+    (title "Hat Labs Marine Engine & Tank interface (HALMET)")
+    (date "2023-11-27")
+    (rev "1.0.0")
     (company "Hat Labs Ltd")
     (comment 1 "https://creativecommons.org/licenses/by-sa/4.0")

Commit message: Update parts according to availability
Parts:
- D1001, D1002: LCSC C72043 -> C965804
- D501: LCSC C72041 -> C84266
Changed lines of the file:
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@@
       (effects (font (size 1.27 1.27)) hide)
     )
-    (property "LCSC" "C72041" (at 44.45 46.99 0)
+    (property "LCSC" "C84266" (at 44.45 46.99 0)
       (effects (font (size 1.27 1.27)) hide)
     )
@@
       (effects (font (size 1.27 1.27)) hide)
     )
-    (property "LCSC" "C72043" (at 93.98 46.99 0)
+    (property "LCSC" "C965804" (at 93.98 46.99 0)
       (effects (font (size 1.27 1.27)) hide)
     )
@@
       (effects (font (size 1.27 1.27)) hide)
     )
-    (property "LCSC" "C72043" (at 78.74 46.99 0)
-      (effects (font (size 1.27 1.27)) hide)
-    )
+    (property "LCSC" "C965804" (at 78.74 46.99 0)
+      (effects (font (size 1.27 1.27)) hide)
+    )
