File: USB.kicad_sch (KiCad schematic)
At the start: 15 parts, among them J401 USB_B_Micro, Q401 S8050, Q402 S8050, U401 CH340C

Commit message: HALMET redesign
Parts:
- added C1002: 100nF, Capacitor_SMD:C_0402_1005Metric, symbol Device:C
- C403, C404: now left out of the parts list
- J401: symbol SH-ESP32:USB_B_Micro-Connector -> HALMET:USB_B_Micro-Connector
- Q401, Q402: symbol SH-ESP32:S8050 -> HALMET:S8050
Connections:
- net GND: now also C1002.2
- net +3V3 renamed +3.3V
- net +3.3V: now also C1002.1
Other:
- title: Sailor Hat with ESP32 -> Hat Labs Marine Engine/Tank interface (HALMET)
Changed lines of the file:
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@@
   (paper "A4")
   (title_block
-    (title "Sailor Hat with ESP32")
-    (date "2023-08-10")
-    (rev "2.0.3")
+    (title "Hat Labs Marine Engine/Tank interface (HALMET)")
+    (date "2023-09-19")
+    (rev "1.0.0-a1")
     (company "Hat Labs Ltd")
     (comment 1 "https://creativecommons.org/licenses/by-sa/4.0")
     (comment 2 "To view a copy of this license, visit ")
-    (comment 3 "SH-ESP32 is licensed under CC BY-SA 4.0.")
+    (comment 3 "HALMET is licensed under CC BY-SA 4.0.")
   )
   (junction (at 52.07 95.25) (diameter 0) (color 0 0 0 0)
@@
     (effects (font (size 1.27 1.27)) (justify left))
   )
-  (symbol (lib_id "SH-ESP32:USB_B_Micro-Connector") (at 25.4 44.45 0) (unit 1)
+  (symbol (lib_id "HALMET:USB_B_Micro-Connector") (at 25.4 44.45 0) (unit 1)
     (in_bom yes) (on_board yes) (dnp no)
     (property "Reference" "J401" (at 26.8478 32.5882 0)
@@
     (pin "6")
     (instances
-      (project "SH-ESP32"
+      (project "HALMET"
         (path "/dff502f1-2fe5-4c09-a767-aabc78c2e052/00000000-0000-0000-0000-00005f89c30a"
           (reference "J401") (unit 1)
@@
     (pin "1")
     (instances
-      (project "SH-ESP32"
+      (project "HALMET"
         (path "/dff502f1-2fe5-4c09-a767-aabc78c2e052/00000000-0000-0000-0000-00005f89c30a"
           (reference "#PWR0402") (unit 1)
@@
     (pin "2")
     (instances
-      (project "SH-ESP32"
+      (project "HALMET"
         (path "/dff502f1-2fe5-4c09-a767-aabc78c2e052/00000000-0000-0000-0000-00005f89c30a"
           (reference "R401") (unit 1)
@@
     (pin "2")
     (instances
-      (project "SH-ESP32"
+      (project "HALMET"
         (path "/dff502f1-2fe5-4c09-a767-aabc78c2e052/00000000-0000-0000-0000-00005f89c30a"
           (reference "R402") (unit 1)
@@
     (pin "9")
     (instances
-      (project "SH-ESP32"
+      (project "HALMET"
         (path "/dff502f1-2fe5-4c09-a767-aabc78c2e052/00000000-0000-0000-0000-00005f89c30a"
           (reference "U401") (unit 1)
@@
     )
   )
-  (symbol (lib_id "SH-ESP32:S8050") (at 130.81 101.6 0) (unit 1)
+  (symbol (lib_id "HALMET:S8050") (at 130.81 101.6 0) (unit 1)
     (in_bom yes) (on_board yes) (dnp no)
     (property "Reference" "Q401" (at 135.636 100.4316 0)
@@
     (pin "3")
     (instances
-      (project "SH-ESP32"
+      (project "HALMET"
         (path "/dff502f1-2fe5-4c09-a767-aabc78c2e052/00000000-0000-0000-0000-00005f89c30a"
           (reference "Q401") (unit 1)
@@
     )
   )
-  (symbol (lib_id "SH-ESP32:S8050") (at 130.81 120.65 0) (mirror x) (unit 1)
+  (symbol (lib_id "HALMET:S8050") (at 130.81 120.65 0) (mirror x) (unit 1)
     (in_bom yes) (on_board yes) (dnp no)
     (property "Reference" "Q402" (at 135.636 119.4816 0)
@@
     (pin "3")
     (instances
-      (project "SH-ESP32"
+      (project "HALMET"
         (path "/dff502f1-2fe5-4c09-a767-aabc78c2e052/00000000-0000-0000-0000-00005f89c30a"
           (reference "Q402") (unit 1)
@@
     (pin "2")
     (instances
-      (project "SH-ESP32"
+      (project "HALMET"
         (path "/dff502f1-2fe5-4c09-a767-aabc78c2e052/00000000-0000-0000-0000-00005f89c30a"
           (reference "C402") (unit 1)
@@
     (pin "1")
     (instances
-      (project "SH-ESP32"
+      (project "HALMET"
         (path "/dff502f1-2fe5-4c09-a767-aabc78c2e052/00000000-0000-0000-0000-00005f89c30a"
           (reference "#PWR0405") (unit 1)
@@
     (pin "1")
     (instances
-      (project "SH-ESP32"
+      (project "HALMET"
         (path "/dff502f1-2fe5-4c09-a767-aabc78c2e052/00000000-0000-0000-0000-00005f89c30a"
           (reference "#PWR0404") (unit 1)
@@
     (pin "2")
     (instances
-      (project "SH-ESP32"
+      (project "HALMET"
         (path "/dff502f1-2fe5-4c09-a767-aabc78c2e052/00000000-0000-0000-0000-00005f89c30a"
           (reference "FB401") (unit 1)
@@
   )
   (symbol (lib_id "Device:C") (at 114.3 52.07 0) (unit 1)
-    (in_bom yes) (on_board yes) (dnp no)
+    (in_bom no) (on_board yes) (dnp no)
     (property "Reference" "C403" (at 117.221 50.9016 0)
       (effects (font (size 1.27 1.27)) (justify left))
@@
     (pin "2")
     (instances
-      (project "SH-ESP32"
+      (project "HALMET"
         (path "/dff502f1-2fe5-4c09-a767-aabc78c2e052/00000000-0000-0000-0000-00005f89c30a"
           (reference "C403") (unit 1)
@@
   )
   (symbol (lib_id "Device:C") (at 127 49.53 0) (unit 1)
-    (in_bom yes) (on_board yes) (dnp no)
+    (in_bom no) (on_board yes) (dnp no)
     (property "Reference" "C404" (at 129.921 48.3616 0)
       (effects (font (size 1.27 1.27)) (justify left))
@@
     (pin "2")
     (instances
-      (project "SH-ESP32"
+      (project "HALMET"
         (path "/dff502f1-2fe5-4c09-a767-aabc78c2e052/00000000-0000-0000-0000-00005f89c30a"
           (reference "C404") (unit 1)
@@
     (pin "1")
     (instances
-      (project "SH-ESP32"
+      (project "HALMET"
         (path "/dff502f1-2fe5-4c09-a767-aabc78c2e052/00000000-0000-0000-0000-00005f89c30a"
           (reference "#PWR0407") (unit 1)
@@
     (pin "1")
     (instances
-      (project "SH-ESP32"
+      (project "HALMET"
         (path "/dff502f1-2fe5-4c09-a767-aabc78c2e052/00000000-0000-0000-0000-00005f89c30a"
           (reference "#PWR0408") (unit 1)
@@
     (pin "2")
     (instances
-      (project "SH-ESP32"
+      (project "HALMET"
         (path "/dff502f1-2fe5-4c09-a767-aabc78c2e052/00000000-0000-0000-0000-00005f89c30a"
           (reference "F401") (unit 1)
@@
     (pin "1")
     (instances
-      (project "SH-ESP32"
+      (project "HALMET"
         (path "/dff502f1-2fe5-4c09-a767-aabc78c2e052/00000000-0000-0000-0000-00005f89c30a"
           (reference "#PWR0109") (unit 1)
@@
     (pin "2")
     (instances
-      (project "SH-ESP32"
+      (project "HALMET"
         (path "/dff502f1-2fe5-4c09-a767-aabc78c2e052/00000000-0000-0000-0000-00005f89c30a"
           (reference "C503") (unit 1)
@@
     (pin "1")
     (instances
-      (project "SH-ESP32"
+      (project "HALMET"
         (path "/dff502f1-2fe5-4c09-a767-aabc78c2e052/00000000-0000-0000-0000-00005f89c30a"
           (reference "#PWR0506") (unit 1)
@@
     )
   )
+  (symbol (lib_id "power:GND") (at 63.5 104.14 0) (unit 1)
+    (in_bom yes) (on_board yes) (dnp no)
+    (property "Reference" "#PWR0901" (at 63.5 110.49 0)
+      (effects (font (size 1.27 1.27)) hide)
+    )
+    (property "Value" "GND" (at 63.627 108.5342 0)
+      (effects (font (size 1.27 1.27)))
+    )
+    (property "Footprint" "" (at 63.5 104.14 0)
+      (effects (font (size 1.27 1.27)) hide)
+    )
+    (property "Datasheet" "" (at 63.5 104.14 0)
+      (effects (font (size 1.27 1.27)) hide)
+    )
+    (pin "1")
+    (instances
+      (project "HALMET"
+        (path "/dff502f1-2fe5-4c09-a767-aabc78c2e052/00000000-0000-0000-0000-00005f89c30a"
+          (reference "#PWR0901") (unit 1)
+        )
+      )
+    )
+  )
   (symbol (lib_id "power:GND") (at 97.79 67.31 0) (unit 1)
     (in_bom yes) (on_board yes) (dnp no)
@@
     (pin "1")
     (instances
-      (project "SH-ESP32"
+      (project "HALMET"
         (path "/dff502f1-2fe5-4c09-a767-aabc78c2e052/00000000-0000-0000-0000-00005f89c30a"
           (reference "#PWR0906") (unit 1)
+        )
+      )
+    )
+  )
+  (symbol (lib_id "Device:C") (at 63.5 100.33 0) (mirror y) (unit 1)
+    (in_bom yes) (on_board yes) (dnp no)
+    (property "Reference" "C1002" (at 60.96 99.06 0)
+      (effects (font (size 1.27 1.27)) (justify left))
+    )
+    (property "Value" "100nF" (at 60.96 101.6 0)
+      (effects (font (size 1.27 1.27)) (justify left))
+    )
+    (property "Footprint" "Capacitor_SMD:C_0402_1005Metric" (at 62.5348 104.14 0)
+      (effects (font (size 1.27 1.27)) hide)
+    )
+    (property "Datasheet" "~" (at 63.5 100.33 0)
+      (effects (font (size 1.27 1.27)) hide)
+    )
+    (property "LCSC" "C1525" (at 63.5 100.33 0)
+      (effects (font (size 1.27 1.27)) hide)
+    )
+    (property "JLCPCB_CORRECTION" "" (at 63.5 100.33 0)
+      (effects (font (size 1.27 1.27)) hide)
+    )
+    (pin "1")
+    (pin "2")
+    (instances
+      (project "HALMET"
+        (path "/dff502f1-2fe5-4c09-a767-aabc78c2e052/00000000-0000-0000-0000-00005fc0c355"
+          (reference "C1002") (unit 1)
+        )
+        (path "/dff502f1-2fe5-4c09-a767-aabc78c2e052/00000000-0000-0000-0000-00005f89c30a"
+          (reference "C901") (unit 1)
         )
       )
@@
     (pin "2")
     (instances
-      (project "SH-ESP32"
+      (project "HALMET"
         (path "/dff502f1-2fe5-4c09-a767-aabc78c2e052/00000000-0000-0000-0000-00005f89c30a"
           (reference "D904") (unit 1)
@@
     (pin "2")
     (instances
-      (project "SH-ESP32"
+      (project "HALMET"
         (path "/dff502f1-2fe5-4c09-a767-aabc78c2e052/00000000-0000-0000-0000-00005f89c30a"
           (reference "D905") (unit 1)
@@
     (pin "1")
     (instances
-      (project "SH-ESP32"
+      (project "HALMET"
         (path "/dff502f1-2fe5-4c09-a767-aabc78c2e052/00000000-0000-0000-0000-00005f89c30a"
           (reference "#PWR0904") (unit 1)
@@
     (pin "2")
     (instances
-      (project "SH-ESP32"
+      (project "HALMET"
         (path "/dff502f1-2fe5-4c09-a767-aabc78c2e052/00000000-0000-0000-0000-00005f89c30a"
           (reference "D903") (unit 1)
@@
     (pin "1")
     (instances
-      (project "SH-ESP32"
+      (project "HALMET"
         (path "/dff502f1-2fe5-4c09-a767-aabc78c2e052/00000000-0000-0000-0000-00005f89c30a"
           (reference "#PWR0905") (unit 1)

Commit message: Implement HALMET v1.0.0 design changes
Other:
- title: Hat Labs Marine Engine/Tank interface (HALMET) -> Hat Labs Marine Engine & Tank interface (HALMET)
Changed lines of the file:
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@@
   (paper "A4")
   (title_block
-    (title "Hat Labs Marine Engine/Tank interface (HALMET)")
-    (date "2023-09-19")
-    (rev "1.0.0-a1")
+    (title "Hat Labs Marine Engine & Tank interface (HALMET)")
+    (date "2023-11-27")
+    (rev "1.0.0")
     (company "Hat Labs Ltd")
     (comment 1 "https://creativecommons.org/licenses/by-sa/4.0")

Commit message: Update parts according to availability
Parts:
- F401: value ASMD1206-050 -> BSMD1206-100-6V; LCSC C135338 -> C883129
Changed lines of the file:
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@@
       (effects (font (size 1.27 1.27)))
     )
-    (property "Value" "ASMD1206-050" (at 48.26 36.6776 90)
+    (property "Value" "BSMD1206-100-6V" (at 48.26 36.6776 90)
       (effects (font (size 1.27 1.27)))
     )
@@
       (effects (font (size 1.27 1.27)) hide)
     )
-    (property "Datasheet" "https://datasheet.lcsc.com/szlcsc/Shenzhen-JDT-Fuse-ASMD1206-050_C135338.pdf" (at 48.26 39.37 0)
+    (property "Datasheet" "https://datasheet.lcsc.com/lcsc/2305121423_BHFUSE-BSMD1206-100-6V_C883129.pdf" (at 48.26 39.37 0)
       (effects (font (size 1.27 1.27)) hide)
     )
-    (property "LCSC" "C135338" (at 48.26 39.37 0)
+    (property "LCSC" "C883129" (at 48.26 39.37 0)
       (effects (font (size 1.27 1.27)) hide)
     )

Commit message: Save with a newer KiCad; change parts for availability; fix rotations
Parts:
- renumbered C1002 to C901
