File: analog_input.kicad_sch (KiCad schematic)
At the start: 60 parts, among them J602 Conn_02x04_Odd_Even, J604 Conn_01x02, J605 Conn_01x02, J606 Conn_01x02, J607 Conn_01x02, Q601 S9015, Q602 S9015, Q603 S9015, Q604 S9015, U601 LMV324, U602 ADS1115IDGS

Commit message: Substitute parts according to availability
Parts:
- Q601, Q602, Q603, Q604: LCSC C106811 -> C5240616; Notes (none) -> Alt: C106811
Changed lines of the file:
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@@
       (effects (font (size 1.27 1.27)) hide)
     )
-    (property "LCSC" "C106811" (at 135.89 55.88 0)
+    (property "LCSC" "C5240616" (at 135.89 55.88 0)
+      (effects (font (size 1.27 1.27)) hide)
+    )
+    (property "Notes" "Alt: C106811" (at 135.89 55.88 0)
       (effects (font (size 1.27 1.27)) hide)
     )
@@
       (effects (font (size 1.27 1.27)) hide)
     )
-    (property "LCSC" "C106811" (at 135.89 95.25 0)
+    (property "LCSC" "C5240616" (at 135.89 95.25 0)
+      (effects (font (size 1.27 1.27)) hide)
+    )
+    (property "Notes" "Alt: C106811" (at 135.89 95.25 0)
       (effects (font (size 1.27 1.27)) hide)
     )
@@
       (effects (font (size 1.27 1.27)) hide)
     )
-    (property "LCSC" "C106811" (at 135.89 133.35 0)
+    (property "LCSC" "C5240616" (at 135.89 133.35 0)
+      (effects (font (size 1.27 1.27)) hide)
+    )
+    (property "Notes" "Alt: C106811" (at 135.89 133.35 0)
       (effects (font (size 1.27 1.27)) hide)
     )
@@
       (effects (font (size 1.27 1.27)) hide)
     )
-    (property "LCSC" "C106811" (at 135.89 168.91 0)
-      (effects (font (size 1.27 1.27)) hide)
-    )
+    (property "LCSC" "C5240616" (at 135.89 168.91 0)
+      (effects (font (size 1.27 1.27)) hide)
+    )
+    (property "Notes" "Alt: C106811" (at 135.89 168.91 0)
+      (effects (font (size 1.27 1.27)) hide)
+    )

Commit message: Implement HALMET v1.0.0 design changes
Parts:
- D603, D604, D605, D611, Q601, Q602, Q603, Q604: JLCPCB_CORRECTION (none) -> 0;0;180
- J602: JLCPCB_CORRECTION (none) -> 1.27;3.81;90
- J604, J605, J606, J607: LCSC C8466 -> C8396
- R613, R614, R616, R618: footprint Resistor_SMD:R_0402_1005Metric -> Resistor_SMD:R_0603_1608Metric; LCSC C25765 -> C4184
- U601, U602: JLCPCB_CORRECTION (none) -> 0;0;270
Other:
- title: Hat Labs Marine Engine/Tank interface (HALMET) -> Hat Labs Marine Engine & Tank interface (HALMET)
Changed lines of the file:
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@@
   (paper "A4")
   (title_block
-    (title "Hat Labs Marine Engine/Tank interface (HALMET)")
-    (date "2023-09-19")
-    (rev "1.0.0-a1")
+    (title "Hat Labs Marine Engine & Tank interface (HALMET)")
+    (date "2023-11-27")
+    (rev "1.0.0")
     (company "Hat Labs Ltd")
     (comment 1 "https://creativecommons.org/licenses/by-sa/4.0")
@@
       (effects (font (size 1.27 1.27)) hide)
     )
+    (property "JLCPCB_CORRECTION" "0;0;270" (at 120.65 95.25 0)
+      (effects (font (size 1.27 1.27)) hide)
+    )
     (pin "1")
     (pin "2")
@@
       (effects (font (size 1.27 1.27)) hide)
     )
+    (property "JLCPCB_CORRECTION" "0;0;270" (at 120.65 168.91 0)
+      (effects (font (size 1.27 1.27)) hide)
+    )
     (pin "1")
     (pin "2")
@@
       (effects (font (size 1.27 1.27)) hide)
     )
+    (property "JLCPCB_CORRECTION" "0;0;270" (at 120.65 133.35 0)
+      (effects (font (size 1.27 1.27)) hide)
+    )
     (pin "1")
     (pin "2")
@@
       (effects (font (size 1.27 1.27)) hide)
     )
+    (property "JLCPCB_CORRECTION" "0;0;270" (at 120.65 55.88 0)
+      (effects (font (size 1.27 1.27)) hide)
+    )
     (pin "1")
     (pin "2")
@@
       (effects (font (size 1.27 1.27)) hide)
     )
+    (property "JLCPCB_CORRECTION" "0;0;270" (at 166.37 165.1 0)
+      (effects (font (size 1.27 1.27)) hide)
+    )
     (pin "1")
     (pin "2")
@@
       (effects (font (size 1.27 1.27)) hide)
     )
+    (property "JLCPCB_CORRECTION" "0;0;180" (at 135.89 55.88 0)
+      (effects (font (size 1.27 1.27)) hide)
+    )
     (pin "1")
     (pin "2")
@@
       (effects (font (size 1.27 1.27)))
     )
-    (property "Footprint" "Resistor_SMD:R_0402_1005Metric" (at 197.358 33.02 90)
+    (property "Footprint" "Resistor_SMD:R_0603_1608Metric" (at 197.358 33.02 90)
       (effects (font (size 1.27 1.27)) hide)
     )
@@
       (effects (font (size 1.27 1.27)) hide)
     )
-    (property "LCSC" "C25765" (at 195.58 33.02 0)
+    (property "LCSC" "C4184" (at 195.58 33.02 0)
       (effects (font (size 1.27 1.27)) hide)
     )
@@
       (effects (font (size 1.27 1.27)) hide)
     )
+    (property "JLCPCB_CORRECTION" "0;0;180" (at 135.89 95.25 0)
+      (effects (font (size 1.27 1.27)) hide)
+    )
     (pin "1")
     (pin "2")
@@
       (effects (font (size 1.27 1.27)) hide)
     )
+    (property "JLCPCB_CORRECTION" "0;0;180" (at 135.89 133.35 0)
+      (effects (font (size 1.27 1.27)) hide)
+    )
     (pin "1")
     (pin "2")
@@
       (effects (font (size 1.27 1.27)) hide)
     )
+    (property "JLCPCB_CORRECTION" "0;0;180" (at 135.89 168.91 0)
+      (effects (font (size 1.27 1.27)) hide)
+    )
     (pin "1")
     (pin "2")
@@
       (effects (font (size 1.27 1.27)) hide)
     )
+    (property "JLCPCB_CORRECTION" "0;0;270" (at 254 74.93 0)
+      (effects (font (size 1.27 1.27)) hide)
+    )
     (pin "1")
     (pin "10")
@@
       (effects (font (size 1.27 1.27)) hide)
     )
+    (property "JLCPCB_CORRECTION" "1.27;3.81;90" (at 73.66 184.15 0)
+      (effects (font (size 1.27 1.27)) hide)
+    )
     (pin "1")
     (pin "2")
@@
       (effects (font (size 1.27 1.27)) hide)
     )
-    (property "LCSC" "C8466" (at 35.56 44.45 0)
+    (property "LCSC" "C8396" (at 35.56 44.45 0)
       (effects (font (size 1.27 1.27)) hide)
     )
@@
       (effects (font (size 1.27 1.27)) hide)
     )
+    (property "JLCPCB_CORRECTION" "0;0;180" (at 214.63 38.1 0)
+      (effects (font (size 1.27 1.27)) hide)
+    )
     (pin "1")
     (pin "2")
@@
       (effects (font (size 1.27 1.27)))
     )
-    (property "Footprint" "Resistor_SMD:R_0402_1005Metric" (at 197.358 59.69 90)
+    (property "Footprint" "Resistor_SMD:R_0603_1608Metric" (at 197.358 59.69 90)
       (effects (font (size 1.27 1.27)) hide)
     )
@@
       (effects (font (size 1.27 1.27)) hide)
     )
-    (property "LCSC" "C25765" (at 195.58 59.69 0)
+    (property "LCSC" "C4184" (at 195.58 59.69 0)
       (effects (font (size 1.27 1.27)) hide)
     )
@@
       (effects (font (size 1.27 1.27)) hide)
     )
-    (property "LCSC" "C8466" (at 35.56 29.21 0)
+    (property "LCSC" "C8396" (at 35.56 29.21 0)
       (effects (font (size 1.27 1.27)) hide)
     )
@@
       (effects (font (size 1.27 1.27)) hide)
     )
+    (property "JLCPCB_CORRECTION" "0;0;180" (at 214.63 118.11 0)
+      (effects (font (size 1.27 1.27)) hide)
+    )
     (pin "1")
     (pin "2")
@@
       (effects (font (size 1.27 1.27)) hide)
     )
+    (property "JLCPCB_CORRECTION" "0;0;180" (at 214.63 91.44 0)
+      (effects (font (size 1.27 1.27)) hide)
+    )
     (pin "1")
     (pin "2")
@@
       (effects (font (size 1.27 1.27)))
     )
-    (property "Footprint" "Resistor_SMD:R_0402_1005Metric" (at 197.358 113.03 90)
+    (property "Footprint" "Resistor_SMD:R_0603_1608Metric" (at 197.358 113.03 90)
       (effects (font (size 1.27 1.27)) hide)
     )
@@
       (effects (font (size 1.27 1.27)) hide)
     )
-    (property "LCSC" "C25765" (at 195.58 113.03 0)
+    (property "LCSC" "C4184" (at 195.58 113.03 0)
       (effects (font (size 1.27 1.27)) hide)
     )
@@
       (effects (font (size 1.27 1.27)) hide)
     )
-    (property "LCSC" "C8466" (at 35.56 36.83 0)
+    (property "LCSC" "C8396" (at 35.56 36.83 0)
       (effects (font (size 1.27 1.27)) hide)
     )
@@
       (effects (font (size 1.27 1.27)) hide)
     )
-    (property "LCSC" "C8466" (at 35.56 52.07 0)
+    (property "LCSC" "C8396" (at 35.56 52.07 0)
       (effects (font (size 1.27 1.27)) hide)
     )
@@
       (effects (font (size 1.27 1.27)))
     )
-    (property "Footprint" "Resistor_SMD:R_0402_1005Metric" (at 197.358 86.36 90)
+    (property "Footprint" "Resistor_SMD:R_0603_1608Metric" (at 197.358 86.36 90)
       (effects (font (size 1.27 1.27)) hide)
     )
@@
       (effects (font (size 1.27 1.27)) hide)
     )
-    (property "LCSC" "C25765" (at 195.58 86.36 0)
+    (property "LCSC" "C4184" (at 195.58 86.36 0)
       (effects (font (size 1.27 1.27)) hide)
     )
@@
       (effects (font (size 1.27 1.27)) hide)
     )
+    (property "JLCPCB_CORRECTION" "0;0;180" (at 214.63 64.77 0)
+      (effects (font (size 1.27 1.27)) hide)
+    )

Commit message: Save with a newer KiCad; change parts for availability; fix rotations
Parts:
- J604, J605, J606, J607: JLCPCB_CORRECTION (none) -> 1.905;0;180
- Q601, Q602, Q603, Q604: value S9015 -> BC856BW,115; LCSC C5240616 -> C28063
- renumbered C705 to C601, C702 to C603, C705 to C604, C702 to C605, C705 to C612, C702 to C613, C705 to C614, C702 to C615, FB702 to FB601, FB702 to FB602, FB702 to FB603, FB702 to FB604
