File: canbus.kicad_sch (KiCad schematic)
At the start: 21 parts, among them J501 Conn_01x02, J601 Conn_01x04, U501 SN65HVD230DR, U502 ADuM1201AR, U603 MST5633BTE

Commit message: HALMET redesign
Parts:
- removed C504, C604: 100nF, Capacitor_SMD:C_0402_1005Metric, symbol Device:C
- removed C601: 10nF/50V, Capacitor_SMD:C_0402_1005Metric, symbol Device:C
- removed C603: 10uF/50V, Capacitor_SMD:C_1206_3216Metric, symbol Device:C
- removed C605: 10uF/10V, Capacitor_SMD:C_0603_1608Metric, symbol Device:C
- removed D202: SM24CANB, Package_TO_SOT_SMD:SOT-23, symbol Device:D_TVS_Dual_AAC
- removed D601: SMBJ33CA, Diode_SMD:D_SMB, symbol Device:D_TVS
- removed D602: B5819W, Diode_SMD:D_SOD-123, symbol Device:D_Schottky
- removed F601: mSMD050-60V, Fuse:Fuse_1812_4532Metric, symbol Device:Polyfuse
- removed FB601: GZ2012D601TF, Inductor_SMD:L_0805_2012Metric, symbol Device:FerriteBead
- removed J501: Conn_01x02, Connector_PinHeader_2.54mm:PinHeader_1x02_P2.54mm_Vertical, symbol Connector_Generic:Conn_01x02
- removed J601: Conn_01x04, Connector_Phoenix_MC:PhoenixContact_MCV_1,5_4-G-3.81_1x04_P3.81mm_Vertical, symbol Connector_Generic:Conn_01x04
- removed U502: ADuM1201AR, Package_SO:SOIC-8_3.9x4.9mm_P1.27mm, symbol Isolator:ADuM1201AR
- removed U603: MST5633BTE, Package_TO_SOT_SMD:SOT-23, symbol SH-ESP32:HT75xx-1-SOT23
- JP601: footprint SH-ESP32:SolderJumper-2_P1.3mm_Open_TrianglePad_Narrow -> HALMET:SolderJumper-2_P1.3mm_Open_TrianglePad_Narrow
Connections:
- net CAN_3V3 is gone; now on net +3.3V: C602.1, U501.3 (VCC)
- net CAN_GND is gone; now on net GND: C602.2, R503.2, U501.2 (GND)
- net D is gone; now on net CAN_TX: U501.1 (D)
- net R is gone; now on net CAN_RX: U501.4 (R)
- net +3V3 renamed +3.3V
Other:
- note removed: "3.3V power feed for the bus side of the CAN bus tranceiver"
- note removed: "Alternatives: - H7533-H#"
- note removed: "Input voltage up to 35V. Output current at least 100mA."
- note removed: "NMEA 2000"
- note removed: "WIRE-LINK from CAN12V_Prot to Vin_Prot"
- title: Sailor Hat with ESP32 -> Hat Labs Marine Engine/Tank interface (HALMET)
- moved on the sheet: R213

Commit message: Implement HALMET v1.0.0 design changes
Other:
- title: Hat Labs Marine Engine/Tank interface (HALMET) -> Hat Labs Marine Engine & Tank interface (HALMET)
Changed lines of the file:
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@@
   (paper "A4")
   (title_block
-    (title "Hat Labs Marine Engine/Tank interface (HALMET)")
-    (date "2023-09-19")
-    (rev "1.0.0-a1")
+    (title "Hat Labs Marine Engine & Tank interface (HALMET)")
+    (date "2023-11-27")
+    (rev "1.0.0")
     (company "Hat Labs Ltd")
     (comment 1 "https://creativecommons.org/licenses/by-sa/4.0")
