File: isolation.kicad_sch (KiCad schematic)
At the start: 19 parts, among them U1201 pi140U30, U1202 ISO1540, U603 XC6206P332MR

Commit message: Substitute parts according to availability
Parts:
- U1201: value pi140U30 -> π140U30
Changed lines of the file:
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@@
       (effects (font (size 1.27 1.27)))
     )
-    (property "Value" "pi140U30" (at 101.6 96.52 0)
+    (property "Value" "π140U30" (at 101.6 96.52 0)
       (effects (font (size 1.27 1.27)))
     )

Commit message: Implement HALMET v1.0.0 design changes
Parts:
- U1201, U1202: JLCPCB_CORRECTION (none) -> 0;0;270
- U603: JLCPCB_CORRECTION (none) -> 0;0;180
Other:
- title: Hat Labs Marine Engine/Tank interface (HALMET) -> Hat Labs Marine Engine & Tank interface (HALMET)
Changed lines of the file:
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@@
   (paper "A4")
   (title_block
-    (title "Hat Labs Marine Engine/Tank interface (HALMET)")
-    (date "2023-09-19")
-    (rev "1.0.0-a1")
+    (title "Hat Labs Marine Engine & Tank interface (HALMET)")
+    (date "2023-11-27")
+    (rev "1.0.0")
     (company "Hat Labs Ltd")
     (comment 1 "https://creativecommons.org/licenses/by-sa/4.0")
@@
       (effects (font (size 1.27 1.27)) hide)
     )
+    (property "JLCPCB_CORRECTION" "0;0;180" (at 151.13 63.5 0)
+      (effects (font (size 1.27 1.27)) hide)
+    )
     (pin "1")
     (pin "2")
@@
     )
     (property "LCSC" "C179739" (at 101.6 158.75 0)
+      (effects (font (size 1.27 1.27)) hide)
+    )
+    (property "JLCPCB_CORRECTION" "0;0;270" (at 101.6 158.75 0)
       (effects (font (size 1.27 1.27)) hide)
     )
@@
       (effects (font (size 1.27 1.27)) hide)
     )
+    (property "JLCPCB_CORRECTION" "0;0;270" (at 101.6 114.3 0)
+      (effects (font (size 1.27 1.27)) hide)
+    )

Commit message: Version 1.0.1 changes
- Add a power header to isolated side
- Fix GPIO silk screen bugs
- Add labels for isolated I2C pads
- Bump version to 1.0.1
Parts:
- added J1201: Conn_01x02, Connector_PinHeader_2.54mm:PinHeader_1x02_P2.54mm_Vertical, symbol Connector_Generic:Conn_01x02
Connections:
- net +3.3V_1: now also J1201.2 (Pin_2)
- net GND1: now also J1201.1 (Pin_1)
Changed lines of the file:
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@@
   (title_block
     (title "Hat Labs Marine Engine & Tank interface (HALMET)")
-    (date "2023-11-27")
-    (rev "1.0.0")
+    (date "2024-01-18")
+    (rev "1.0.1")
     (company "Hat Labs Ltd")
     (comment 1 "https://creativecommons.org/licenses/by-sa/4.0")
@@
     (stroke (width 0) (type default))
   )
+  (wire (pts (xy 167.64 60.96) (xy 190.5 60.96))
+    (stroke (width 0) (type default))
+  )
   (wire (pts (xy 86.36 72.39) (xy 86.36 66.04))
     (stroke (width 0) (type default))
@@
     (stroke (width 0) (type default))
   )
-  (wire (pts (xy 190.5 60.96) (xy 167.64 60.96))
-    (stroke (width 0) (type default))
-  )
   (wire (pts (xy 77.47 148.59) (xy 77.47 147.32))
     (stroke (width 0) (type default))
@@
     (stroke (width 0) (type default))
   )
+  (wire (pts (xy 166.37 96.52) (xy 166.37 92.71))
+    (stroke (width 0) (type default))
+  )
   (wire (pts (xy 128.27 93.98) (xy 128.27 92.71))
     (stroke (width 0) (type default))
@@
     (stroke (width 0) (type default))
   )
+  (wire (pts (xy 172.72 96.52) (xy 166.37 96.52))
+    (stroke (width 0) (type default))
+  )
   (wire (pts (xy 118.11 60.96) (xy 119.38 60.96))
     (stroke (width 0) (type default))
@@
   )
   (wire (pts (xy 83.82 124.46) (xy 83.82 128.27))
+    (stroke (width 0) (type default))
+  )
+  (wire (pts (xy 172.72 99.06) (xy 166.37 99.06))
+    (stroke (width 0) (type default))
+  )
+  (wire (pts (xy 166.37 99.06) (xy 166.37 101.6))
     (stroke (width 0) (type default))
   )
@@
     )
   )
+  (symbol (lib_id "Connector_Generic:Conn_01x02") (at 177.8 99.06 0) (mirror x) (unit 1)
+    (in_bom yes) (on_board yes) (dnp no) (fields_autoplaced)
+    (property "Reference" "J1201" (at 177.8 90.17 0)
+      (effects (font (size 1.27 1.27)))
+    )
+    (property "Value" "Conn_01x02" (at 177.8 92.71 0)
+      (effects (font (size 1.27 1.27)))
+    )
+    (property "Footprint" "Connector_PinHeader_2.54mm:PinHeader_1x02_P2.54mm_Vertical" (at 177.8 99.06 0)
+      (effects (font (size 1.27 1.27)) hide)
+    )
+    (property "Datasheet" "~" (at 177.8 99.06 0)
+      (effects (font (size 1.27 1.27)) hide)
+    )
+    (pin "1")
+    (pin "2")
+    (instances
+      (project "HALMET"
+        (path "/dff502f1-2fe5-4c09-a767-aabc78c2e052/2a37b9a7-9486-444f-9ef1-0d0aa57a298a"
+          (reference "J1201") (unit 1)
+        )
+      )
+    )
+  )
   (symbol (lib_id "power:GND1") (at 190.5 69.85 0) (unit 1)
-    (in_bom yes) (on_board yes) (dnp no) (fields_autoplaced)
+    (in_bom yes) (on_board yes) (dnp no)
     (property "Reference" "#PWR01207" (at 190.5 76.2 0)
       (effects (font (size 1.27 1.27)) hide)
@@
         (path "/dff502f1-2fe5-4c09-a767-aabc78c2e052/2a37b9a7-9486-444f-9ef1-0d0aa57a298a"
           (reference "#PWR01211") (unit 1)
+        )
+      )
+    )
+  )
+  (symbol (lib_id "power:GND1") (at 166.37 101.6 0) (unit 1)
+    (in_bom yes) (on_board yes) (dnp no)
+    (property "Reference" "#PWR01222" (at 166.37 107.95 0)
+      (effects (font (size 1.27 1.27)) hide)
+    )
+    (property "Value" "GND1" (at 166.37 106.68 0)
+      (effects (font (size 1.27 1.27)))
+    )
+    (property "Footprint" "" (at 166.37 101.6 0)
+      (effects (font (size 1.27 1.27)) hide)
+    )
+    (property "Datasheet" "" (at 166.37 101.6 0)
+      (effects (font (size 1.27 1.27)) hide)
+    )
+    (pin "1")
+    (instances
+      (project "HALMET"
+        (path "/dff502f1-2fe5-4c09-a767-aabc78c2e052/2a37b9a7-9486-444f-9ef1-0d0aa57a298a"
+          (reference "#PWR01222") (unit 1)
         )
       )
@@
         )
       )
+    )
+  )
+  (symbol (lib_id "HALMET:+3.3V_1") (at 166.37 92.71 0) (unit 1)
+    (in_bom yes) (on_board yes) (dnp no) (fields_autoplaced)
+    (property "Reference" "#PWR01223" (at 166.37 96.52 0)
+      (effects (font (size 1.27 1.27)) hide)
+    )
+    (property "Value" "+3.3V_1" (at 166.37 87.63 0)
+      (effects (font (size 1.27 1.27)))
+    )
+    (property "Footprint" "" (at 166.37 92.71 0)
+      (effects (font (size 1.27 1.27)) hide)
+    )
+    (property "Datasheet" "" (at 166.37 92.71 0)
+      (effects (font (size 1.27 1.27)) hide)
+    )
+    (pin "1")
+    (instances
+      (project "HALMET"
+        (path "/dff502f1-2fe5-4c09-a767-aabc78c2e052/2a37b9a7-9486-444f-9ef1-0d0aa57a298a"
+          (reference "#PWR01223") (unit 1)
+        )
+      )

Commit message: Update parts according to availability
Parts:
- C1209: LCSC C1021634 -> C2940747
Changed lines of the file:
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@@
       (effects (font (size 1.27 1.27)) hide)
     )
-    (property "LCSC" "C1021634" (at 101.6 72.39 0)
+    (property "LCSC" "C2940747" (at 101.6 72.39 0)
       (effects (font (size 1.27 1.27)) hide)
     )

Commit message: Save with a newer KiCad; change parts for availability; fix rotations
Parts:
- PS1201: JLCPCB_CORRECTION (none) -> 0;3.81;270
- renumbered C605 to C1203, C602 to C1204, C602 to C1205, C602 to C1206, C602 to C1207, R701 to R1202, R702 to R1203, U603 to U1203
