File: onewire.kicad_sch (KiCad schematic)
At the start: 9 parts, among them J801 Conn_01x03

Commit message: HALMET redesign
Connections:
- net +3V3 renamed +3.3V
Other:
- title: Sailor Hat with ESP32 -> Hat Labs Marine Engine/Tank interface (HALMET)
Changed lines of the file:
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@@
   (paper "A4")
   (title_block
-    (title "Sailor Hat with ESP32")
-    (date "2023-08-10")
-    (rev "2.0.3")
+    (title "Hat Labs Marine Engine/Tank interface (HALMET)")
+    (date "2023-09-19")
+    (rev "1.0.0-a1")
     (company "Hat Labs Ltd")
     (comment 1 "https://creativecommons.org/licenses/by-sa/4.0")
     (comment 2 "To view a copy of this license, visit ")
-    (comment 3 "SH-ESP32 is licensed under CC BY-SA 4.0.")
+    (comment 3 "HALMET is licensed under CC BY-SA 4.0.")
   )
   (junction (at 116.84 59.69) (diameter 0) (color 0 0 0 0)
@@
     (pin "1")
     (instances
-      (project "SH-ESP32"
+      (project "HALMET"
         (path "/dff502f1-2fe5-4c09-a767-aabc78c2e052/00000000-0000-0000-0000-00005faef03b"
           (reference "#PWR0805") (unit 1)
@@
     (pin "2")
     (instances
-      (project "SH-ESP32"
+      (project "HALMET"
         (path "/dff502f1-2fe5-4c09-a767-aabc78c2e052/00000000-0000-0000-0000-00005faef03b"
           (reference "R801") (unit 1)
@@
     (pin "3")
     (instances
-      (project "SH-ESP32"
+      (project "HALMET"
         (path "/dff502f1-2fe5-4c09-a767-aabc78c2e052/00000000-0000-0000-0000-00005faef03b"
           (reference "J801") (unit 1)
@@
     (pin "1")
     (instances
-      (project "SH-ESP32"
+      (project "HALMET"
         (path "/dff502f1-2fe5-4c09-a767-aabc78c2e052/00000000-0000-0000-0000-00005faef03b"
           (reference "#PWR0809") (unit 1)
@@
     (pin "2")
     (instances
-      (project "SH-ESP32"
+      (project "HALMET"
         (path "/dff502f1-2fe5-4c09-a767-aabc78c2e052/00000000-0000-0000-0000-00005faef03b"
           (reference "C803") (unit 1)
@@
     (pin "1")
     (instances
-      (project "SH-ESP32"
+      (project "HALMET"
         (path "/dff502f1-2fe5-4c09-a767-aabc78c2e052/00000000-0000-0000-0000-00005faef03b"
           (reference "#PWR0808") (unit 1)
@@
     (pin "2")
     (instances
-      (project "SH-ESP32"
+      (project "HALMET"
         (path "/dff502f1-2fe5-4c09-a767-aabc78c2e052/00000000-0000-0000-0000-00005faef03b"
           (reference "C801") (unit 1)
@@
     (pin "2")
     (instances
-      (project "SH-ESP32"
+      (project "HALMET"
         (path "/dff502f1-2fe5-4c09-a767-aabc78c2e052/00000000-0000-0000-0000-00005faef03b"
           (reference "FB801") (unit 1)
@@
     (pin "2")
     (instances
-      (project "SH-ESP32"
+      (project "HALMET"
         (path "/dff502f1-2fe5-4c09-a767-aabc78c2e052/00000000-0000-0000-0000-00005faef03b"
           (reference "R802") (unit 1)
@@
     (pin "2")
     (instances
-      (project "SH-ESP32"
+      (project "HALMET"
         (path "/dff502f1-2fe5-4c09-a767-aabc78c2e052/00000000-0000-0000-0000-00005faef03b"
           (reference "C802") (unit 1)
@@
     (pin "1")
     (instances
-      (project "SH-ESP32"
+      (project "HALMET"
         (path "/dff502f1-2fe5-4c09-a767-aabc78c2e052/00000000-0000-0000-0000-00005faef03b"
           (reference "#PWR0807") (unit 1)
@@
     (pin "1")
     (instances
-      (project "SH-ESP32"
+      (project "HALMET"
         (path "/dff502f1-2fe5-4c09-a767-aabc78c2e052/00000000-0000-0000-0000-00005faef03b"
           (reference "#PWR0802") (unit 1)
@@
     (pin "1")
     (instances
-      (project "SH-ESP32"
+      (project "HALMET"
         (path "/dff502f1-2fe5-4c09-a767-aabc78c2e052/00000000-0000-0000-0000-00005faef03b"
           (reference "#PWR0806") (unit 1)
@@
     (pin "2")
     (instances
-      (project "SH-ESP32"
+      (project "HALMET"
         (path "/dff502f1-2fe5-4c09-a767-aabc78c2e052/00000000-0000-0000-0000-00005faef03b"
           (reference "D504") (unit 1)
@@
     (pin "2")
     (instances
-      (project "SH-ESP32"
+      (project "HALMET"
         (path "/dff502f1-2fe5-4c09-a767-aabc78c2e052/00000000-0000-0000-0000-00005faef03b"
           (reference "D503") (unit 1)
@@
     (pin "1")
     (instances
-      (project "SH-ESP32"
+      (project "HALMET"
         (path "/dff502f1-2fe5-4c09-a767-aabc78c2e052/00000000-0000-0000-0000-00005faef03b"
           (reference "#PWR0508") (unit 1)
@@
     (pin "1")
     (instances
-      (project "SH-ESP32"
+      (project "HALMET"
         (path "/dff502f1-2fe5-4c09-a767-aabc78c2e052/00000000-0000-0000-0000-00005faef03b"
           (reference "#PWR0507") (unit 1)

Commit message: Implement HALMET v1.0.0 design changes
Other:
- title: Hat Labs Marine Engine/Tank interface (HALMET) -> Hat Labs Marine Engine & Tank interface (HALMET)
Changed lines of the file:
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@@
   (paper "A4")
   (title_block
-    (title "Hat Labs Marine Engine/Tank interface (HALMET)")
-    (date "2023-09-19")
-    (rev "1.0.0-a1")
+    (title "Hat Labs Marine Engine & Tank interface (HALMET)")
+    (date "2023-11-27")
+    (rev "1.0.0")
     (company "Hat Labs Ltd")
     (comment 1 "https://creativecommons.org/licenses/by-sa/4.0")
