File: power-input.kicad_sch (KiCad schematic)
At the start: 21 parts, among them J204 Conn_01x02, J301 Conn_01x02, U202 XL1509-3.3

Commit message: HALMET redesign
Parts:
- removed C201: 22nF, Capacitor_SMD:C_0402_1005Metric, symbol Device:C_Small
- removed C301: 22uF/35V, Capacitor_SMD:C_1206_3216Metric, symbol Device:C
- removed C302: 10nF/50V, Capacitor_SMD:C_0402_1005Metric, symbol Device:C
- removed C306: 470nF/50V, Capacitor_SMD:C_0805_2012Metric, symbol Device:C
- removed C307: 1uF/50V, Capacitor_SMD:C_0805_2012Metric, symbol Device:C
- removed C308: 4.7uF/50V, Capacitor_SMD:C_1206_3216Metric, symbol Device:C
- removed D302: DSK24 K24, Diode_SMD:D_SOD-123F, symbol Device:D_Schottky
- removed FB301: GZ2012D601TF, Inductor_SMD:L_0805_2012Metric, symbol Device:FerriteBead
- removed J204: Conn_01x02, Connector_PinHeader_2.54mm:PinHeader_1x02_P2.54mm_Vertical, symbol Connector_Generic:Conn_01x02
- removed J301: Conn_01x02, Connector_Phoenix_MC:PhoenixContact_MCV_1,5_2-G-3.81_1x02_P3.81mm_Vertical, symbol Connector_Generic:Conn_01x02
- removed L302: CBC3225T100MR, Inductor_SMD:L_1210_3225Metric, symbol Device:L
- removed R211: 0, Resistor_SMD:R_0402_1005Metric, symbol Device:R_Small
- removed R212: inf, Resistor_SMD:R_0402_1005Metric, symbol Device:R_Small
- removed R304: 4.7R, Resistor_SMD:R_0603_1608Metric, symbol Device:R
- added C707, C708, C709, C710, C711, C712, C714: 10uF/50V, Capacitor_SMD:C_1206_3216Metric, symbol Device:C
- added C713: 4.7nF/50V, Capacitor_SMD:C_0402_1005Metric, symbol Device:C
- added C715: 1uF/50V, Capacitor_SMD:C_0805_2012Metric, symbol Device:C
- added C716: 4.7uF/50V, Capacitor_SMD:C_1206_3216Metric, symbol Device:C
- added D202: SM24CANB, Package_TO_SOT_SMD:SOT-23, symbol Device:D_TVS_Dual_AAC
- added D701: B5819W, Diode_SMD:D_SOD-123F, symbol Device:D_Schottky
- added FB704: GZ2012D601TF, Inductor_SMD:L_0805_2012Metric, symbol Device:FerriteBead
- added J601: Conn_01x04, Connector_Phoenix_MC:PhoenixContact_MCV_1,5_4-G-3.81_1x04_P3.81mm_Vertical, symbol Connector_Generic:Conn_01x04
- added L701: CBC3225T100KR, Inductor_SMD:L_1210_3225Metric, symbol Device:L
- added R703: 4.7R, Resistor_SMD:R_0603_1608Metric, symbol Device:R
- L301: footprint SH-ESP32:SMMS0650-1R0M -> HALMET:SMMS0650-1R0M
- U202: symbol SH-ESP32:XL1509-ADJE1 -> HALMET:XL1509-ADJE1
Connections:
- net FB is gone; now on net +3.3V: U202.3 (FB)
- net GND: now also C707.2, C708.2, C709.2, C710.2, C711.2, C712.2, C713.2, C714.1, C715.1, D202.3 (common), D701.2 (A), J601.1 (Pin_1), R703.1
- net IN: now also C707.1, C708.1, C709.1, C710.1, C711.1, C712.1, FB704.1
- net SW: now also D701.1 (K)
- net Vin_fused: now also F301.1
- net Vin_protected: now also C714.2, L701.1
- net +3V3 renamed +3.3V
- net Vin renamed CAN_+
- net CAN_+: now also J601.2 (Pin_2)
- new net: C713.1, C715.2, C716.1, FB704.2, L701.2
- new net: C716.2, R703.2
- new net CAN_H: D202.1 (A1), J601.3 (Pin_3)
- new net CAN_L: D202.2 (A2), J601.4 (Pin_4)
Other:
- note added: "Bulk input capacitance is implemented with a number of 10uF MLCC caps to manage the cost."
- note added: "Converter IC voltage range 4.5-50V, however, Vin needs to be a bit higher to give some headroom for the PTC fuse and polarity protection diode."
- note added: "First stage HF input filter. Design as per TI SNVA886."
- note added: "NMEA 2000"
- note added: "Second stage input filter for limiting conducted noise emissions at power input lines. Design as per Rohm 62AN101E."
- note removed: "CAN wire link"
- note removed: "Converter IC voltage range 4.5-50V, however, Vin needs to be a bit higher to give some headroom for the PTC fuse."
- note removed: "Input filter for limiting conducted noise emissions at power input lines."
- title: Sailor Hat with ESP32 -> Hat Labs Marine Engine/Tank interface (HALMET)
- moved on the sheet: D201, L301, U202

Commit message: Implement HALMET v1.0.0 design changes
Other:
- title: Hat Labs Marine Engine/Tank interface (HALMET) -> Hat Labs Marine Engine & Tank interface (HALMET)
Changed lines of the file:
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@@
   (paper "A4")
   (title_block
-    (title "Hat Labs Marine Engine/Tank interface (HALMET)")
-    (date "2023-09-19")
-    (rev "1.0.0-a1")
+    (title "Hat Labs Marine Engine & Tank interface (HALMET)")
+    (date "2023-11-27")
+    (rev "1.0.0")
     (company "Hat Labs Ltd")
     (comment 1 "https://creativecommons.org/licenses/by-sa/4.0")

Commit message: Update parts according to availability
Parts:
- D701: footprint Diode_SMD:D_SOD-123F -> Diode_SMD:D_SOD-123
- L701: value CBC3225T100KR -> NLCV32T-100K-PFR; LCSC C90321 -> C74563
Changed lines of the file:
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@@
       (effects (font (size 1.27 1.27)))
     )
-    (property "Value" "CBC3225T100KR" (at 72.39 119.4054 90)
+    (property "Value" "NLCV32T-100K-PFR" (at 72.39 119.4054 90)
       (effects (font (size 1.27 1.27)))
     )
@@
       (effects (font (size 1.27 1.27)) hide)
     )
-    (property "LCSC" "C90321" (at 72.39 121.92 0)
+    (property "LCSC" "C74563" (at 72.39 121.92 0)
       (effects (font (size 1.27 1.27)) hide)
     )
@@
       (effects (font (size 1.27 1.27)) (justify left))
     )
-    (property "Footprint" "Diode_SMD:D_SOD-123F" (at 220.98 111.76 0)
+    (property "Footprint" "Diode_SMD:D_SOD-123" (at 220.98 111.76 0)
       (effects (font (size 1.27 1.27)) hide)
     )

Commit message: Update parts according to availability
Parts:
- L701: value NLCV32T-100K-PFR -> NLCV32T-100K-EFR; LCSC C74563 -> C295195
Changed lines of the file:
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@@
       (effects (font (size 1.27 1.27)))
     )
-    (property "Value" "NLCV32T-100K-PFR" (at 72.39 119.4054 90)
+    (property "Value" "NLCV32T-100K-EFR" (at 72.39 119.4054 90)
       (effects (font (size 1.27 1.27)))
     )
@@
       (effects (font (size 1.27 1.27)) hide)
     )
-    (property "LCSC" "C74563" (at 72.39 121.92 0)
+    (property "LCSC" "C295195" (at 72.39 121.92 0)
       (effects (font (size 1.27 1.27)) hide)
     )

Commit message: Save with a newer KiCad; change parts for availability; fix rotations
Parts:
- D801: renamed from D202; LCSC C970029 -> C41376477
- renumbered J601 to J802
